File: hardware/electrical/indicators.kicad_sch (KiCad schematic)
At the start: 11 parts

Commit message: (eda): add switching buck converter from 12v to 5v
Parts:
- D201, D202, D203, D204: value Blue -> White
Other:
- note added: "Status LED"
- note removed: "Error Signaling LED"
Changed lines of the file:
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@@
 		)
 	)
-	(text "Error Signaling LED"
+	(text "Status LED"
 		(exclude_from_sim no)
 		(at 55.499 48.133 0)
@@
 			)
 		)
-		(property "Value" "Blue"
+		(property "Value" "White"
 			(at 206.756 72.39 0)
 			(effects
@@
 			)
 		)
-		(property "Value" "Blue"
+		(property "Value" "White"
 			(at 206.756 82.55 0)
 			(effects
@@
 			)
 		)
-		(property "Value" "Blue"
+		(property "Value" "White"
 			(at 206.756 62.23 0)
 			(effects
@@
 			)
 		)
-		(property "Value" "Blue"
+		(property "Value" "White"
 			(at 206.756 52.07 0)
 			(effects
